Commit message: add depth support navigation, finally!!! Not super happy but better, needs improvements in cornering

File: src/yahboomcar_description/urdf/MicroROS.urdf (robot description, URDF)
Before this commit: robot micro4.0, 9 links, 8 joints
Joints:
- added joint tof_Joint: type fixed, parent base_link, child depth_link, origin xyz=0.10 0.05 0.06 rpy=0 0 0, axis 0 0 0
